Commit message: AMCL tuning

File: include/lms1xx/urdf/sick_lms1xx.urdf.xacro (robot description, xacro)
@@ -40,5 +40,5 @@
         <geometry>
           <!-- Origin of this mesh is the focal point of the LIDAR. -->
-          <mesh filename="package://srd_pkg/jackal/jackal_description/urdf/accessories/lms1xx/meshes/sick-lms1xx.dae" />
+          <mesh filename="package://srd_pkg/include/lms1xx/meshes/sick-lms1xx.dae" />
         </geometry>
       </visual>

File: jackal/jackal_description/urdf/accessories.urdf.xacro (robot description, xacro)
@@ -15,5 +15,5 @@
   <!-- 2D Lidars -->
   <xacro:include filename="$(find sick_tim)/urdf/sick_tim.urdf.xacro" />
-  <xacro:include filename="$(find srd_pkg)/jackal/jackal_description/urdf/accessories/lms1xx/urdf/sick_lms1xx.urdf.xacro" />
+  <xacro:include filename="$(find srd_pkg)/include/lms1xx/urdf/sick_lms1xx.urdf.xacro" />
   <xacro:include filename="$(find srd_pkg)/jackal/jackal_description/urdf/accessories/sick_lms1xx_inverted_mount.urdf.xacro" />
   <xacro:include filename="$(find srd_pkg)/jackal/jackal_description/urdf/accessories/sick_lms1xx_upright_mount.urdf.xacro" />

File: jackal/jackal_description/urdf/accessories/sick_lms1xx_inverted_mount.urdf.xacro (robot description, xacro)
@@ -26,5 +26,5 @@
 -->
 <robot xmlns:xacro="http://www.ros.org/wiki/xacro">
-  <xacro:include filename="$(find srd_pkg)/jackal/jackal_description/urdf/accessories/lms1xx/urdf/sick_lms1xx.urdf.xacro" />
+  <xacro:include filename="$(find srd_pkg)/include/lms1xx/urdf/sick_lms1xx.urdf.xacro" />
   <xacro:macro name="sick_lms1xx_inverted_mount" params="prefix topic parent_link *origin">
     <xacro:sick_lms1xx frame="${prefix}_laser" topic="${topic}" />

File: jackal/jackal_description/urdf/accessories/sick_lms1xx_upright_mount.urdf.xacro (robot description, xacro)
@@ -26,5 +26,5 @@
 -->
 <robot xmlns:xacro="http://www.ros.org/wiki/xacro">
-  <xacro:include filename="$(find srd_pkg)/jackal/jackal_description/urdf/accessories/lms1xx/urdf/sick_lms1xx.urdf.xacro" />
+  <xacro:include filename="$(find srd_pkg)/include/lms1xx/urdf/sick_lms1xx.urdf.xacro" />
   <xacro:macro name="sick_lms1xx_upright_mount" params="prefix topic parent_link *origin">
     <xacro:sick_lms1xx frame="${prefix}_laser" topic="${topic}" robot_namespace="$(arg namespace)" />
