Commit message: Stand alone jackal

File: jackal/jackal_description/urdf/accessories.urdf.xacro (robot description, xacro)
@@ -10,16 +10,16 @@
   -->
   <!-- Macros to generate standoffs for offset payload mounting. -->
-  <xacro:include filename="$(find jackal_description)/urdf/accessories/standoffs.urdf.xacro" />
+  <xacro:include filename="$(find srd_pkg)/jackal/jackal_description/urdf/accessories/standoffs.urdf.xacro" />
   <!-- This optional plate mounts both the upgraded GPS and the Velodyne 3D LIDAR. -->
-  <xacro:include filename="$(find jackal_description)/urdf/accessories/bridge_plate.urdf.xacro" />
+  <xacro:include filename="$(find srd_pkg)/jackal/jackal_description/urdf/accessories/bridge_plate.urdf.xacro" />
   <!-- 2D Lidars -->
   <xacro:include filename="$(find sick_tim)/urdf/sick_tim.urdf.xacro" />
   <xacro:include filename="$(find lms1xx)/urdf/sick_lms1xx.urdf.xacro" />
-  <xacro:include filename="$(find jackal_description)/urdf/accessories/sick_lms1xx_inverted_mount.urdf.xacro" />
-  <xacro:include filename="$(find jackal_description)/urdf/accessories/sick_lms1xx_upright_mount.urdf.xacro" />
-  <xacro:include filename="$(find jackal_description)/urdf/accessories/hokuyo_utm30.urdf.xacro" />
-  <xacro:include filename="$(find jackal_description)/urdf/accessories/hokuyo_ust10.urdf.xacro" />
-  <xacro:include filename="$(find jackal_description)/urdf/accessories/vlp16_mount.urdf.xacro" />
-  <xacro:include filename="$(find jackal_description)/urdf/accessories/hdl32_mount.urdf.xacro" />
+  <xacro:include filename="$(find srd_pkg)/jackal/jackal_description/urdf/accessories/sick_lms1xx_inverted_mount.urdf.xacro" />
+  <xacro:include filename="$(find srd_pkg)/jackal/jackal_description/urdf/accessories/sick_lms1xx_upright_mount.urdf.xacro" />
+  <xacro:include filename="$(find srd_pkg)/jackal/jackal_description/urdf/accessories/hokuyo_utm30.urdf.xacro" />
+  <xacro:include filename="$(find srd_pkg)/jackal/jackal_description/urdf/accessories/hokuyo_ust10.urdf.xacro" />
+  <xacro:include filename="$(find srd_pkg)/jackal/jackal_description/urdf/accessories/vlp16_mount.urdf.xacro" />
+  <xacro:include filename="$(find srd_pkg)/jackal/jackal_description/urdf/accessories/hdl32_mount.urdf.xacro" />
   <!--
     Add Microstrain IMU. By default the Jackal comes equipped with an IMU linked to "imu_link". These extra
@@ -195,6 +195,6 @@
     - smart7              :: Novatel Smart7
   -->
-  <xacro:include filename="$(find jackal_description)/urdf/accessories/novatel_smart6.urdf.xacro" />
-  <xacro:include filename="$(find jackal_description)/urdf/accessories/novatel_smart7.urdf.xacro" />
+  <xacro:include filename="$(find srd_pkg)/jackal/jackal_description/urdf/accessories/novatel_smart6.urdf.xacro" />
+  <xacro:include filename="$(find srd_pkg)/jackal/jackal_description/urdf/accessories/novatel_smart7.urdf.xacro" />
   <xacro:if value="$(optenv JACKAL_NAVSAT 0)">
     <xacro:property name="mount" value="$(optenv JACKAL_NAVSAT_MOUNT rear)" />
@@ -257,5 +257,5 @@
   -->
   <!-- Common camera mounts and accessory URDFs. -->
-  <xacro:include filename="$(find jackal_description)/urdf/accessories/camera_mount.urdf.xacro" />
+  <xacro:include filename="$(find srd_pkg)/jackal/jackal_description/urdf/accessories/camera_mount.urdf.xacro" />
   <xacro:include filename="$(find pointgrey_camera_description)/urdf/pointgrey_flea3.urdf.xacro" />
   <!-- If enabled, generate the flea3 camera payload with a tilt of 30 degrees. -->
@@ -302,5 +302,5 @@
     </xacro:unless>
   </xacro:if>
-  <xacro:include filename="$(find jackal_description)/urdf/accessories/stereo_camera_mount.urdf.xacro" />
+  <xacro:include filename="$(find srd_pkg)/jackal/jackal_description/urdf/accessories/stereo_camera_mount.urdf.xacro" />
   <!-- If enabled, generates a pair of flea3 cameras for stereo vision with a tilt of 30 degrees. -->
   <!-- Disabled temporarily due to metapackage issue. -->
@@ -396,5 +396,5 @@
   <!-- Fender Accessories -->
   <xacro:if value="$(optenv JACKAL_FRONT_ACCESSORY_FENDER 0)">
-    <xacro:include filename="$(find jackal_description)/urdf/accessories/hokuyo_ust10.urdf.xacro" />
+    <xacro:include filename="$(find srd_pkg)/jackal/jackal_description/urdf/accessories/hokuyo_ust10.urdf.xacro" />
     <xacro:if value="$(optenv JACKAL_FRONT_FENDER_UST10 0)">
       <xacro:hokuyo_ust10_mount
@@ -425,5 +425,5 @@
       <visual>
         <geometry>
-          <mesh filename="package://jackal_description/meshes/wibotic_bumper.stl" />
+          <mesh filename="package://srd_pkg/jackal/jackal_description/meshes/wibotic_bumper.stl" />
         </geometry>
         <material name="dark_grey" />
@@ -447,5 +447,5 @@
         <origin xyz="0 0 0" rpy="0 0 0"/>
         <geometry>
-          <mesh filename="package://jackal_description/meshes/ark_enclosure.stl"/>
+          <mesh filename="package://srd_pkg/jackal/jackal_description/meshes/ark_enclosure.stl"/>
         </geometry>
         <material name="dark_grey" />

File: jackal/jackal_description/urdf/accessories/bridge_plate.urdf.xacro (robot description, xacro)
@@ -17,5 +17,5 @@
         <origin xyz="0 0 0" rpy="1.5707 0.0 1.5707" />
         <geometry>
-          <mesh filename="package://jackal_description/meshes/bridge-plate.stl"/>
+          <mesh filename="package://srd_pkg/jackal/jackal_description/meshes/bridge-plate.stl"/>
         </geometry>
         <material name="dark_grey" />

File: jackal/jackal_description/urdf/accessories/camera_mount.urdf.xacro (robot description, xacro)
@@ -5,5 +5,5 @@
         <origin xyz="0 0 0" rpy="1.5707 0 1.5707" />
         <geometry>
-          <mesh filename="package://jackal_description/meshes/camera-bracket.stl" scale="0.001 0.001 0.001" />
+          <mesh filename="package://srd_pkg/jackal/jackal_description/meshes/camera-bracket.stl" scale="0.001 0.001 0.001" />
         </geometry>
         <material name="dark_grey" />
@@ -14,5 +14,5 @@
         <origin xyz="0 0 0" rpy="0 0 1.5707" />
         <geometry>
-          <mesh filename="package://jackal_description/meshes/camera-beam.stl" scale="0.001 0.001 0.001" />
+          <mesh filename="package://srd_pkg/jackal/jackal_description/meshes/camera-beam.stl" scale="0.001 0.001 0.001" />
         </geometry>
         <material name="dark_grey" />

File: jackal/jackal_description/urdf/accessories/hdl32_mount.urdf.xacro (robot description, xacro)
@@ -6,5 +6,5 @@
         <visual>
           <geometry>
-            <mesh filename="package://jackal_description/meshes/velodyne_tower.stl"/>
+            <mesh filename="package://srd_pkg/jackal/jackal_description/meshes/velodyne_tower.stl"/>
           </geometry>
           <origin xyz="0 0 0" rpy="0 0 0" />
@@ -13,5 +13,5 @@
         <collision>
           <geometry>
-            <mesh filename="package://jackal_description/meshes/velodyne_tower.stl"/>
+            <mesh filename="package://srd_pkg/jackal/jackal_description/meshes/velodyne_tower.stl"/>
           </geometry>
           <origin xyz="0 0 0" rpy="0 0 0" />

File: jackal/jackal_description/urdf/accessories/hokuyo_ust10.urdf.xacro (robot description, xacro)
@@ -58,5 +58,5 @@
         <geometry>
           <!-- Origin of this mesh is the base of the bracket. -->
-          <mesh filename="package://jackal_description/meshes/hokuyo_ust10.stl" />
+          <mesh filename="package://srd_pkg/jackal/jackal_description/meshes/hokuyo_ust10.stl" />
         </geometry>
         <material name="dark_grey" />

File: jackal/jackal_description/urdf/accessories/hokuyo_utm30.urdf.xacro (robot description, xacro)
@@ -61,5 +61,5 @@
         <geometry>
           <!-- Origin of this mesh is the base of the bracket. -->
-          <mesh filename="package://jackal_description/meshes/hokuyo_utm30.stl" />
+          <mesh filename="package://srd_pkg/jackal/jackal_description/meshes/hokuyo_utm30.stl" />
         </geometry>
         <material name="dark_grey" />

File: jackal/jackal_description/urdf/accessories/novatel_smart6.urdf.xacro (robot description, xacro)
@@ -6,5 +6,5 @@
       <origin xyz="0 0 0" rpy="0 0 0" />
       <geometry>
-        <mesh filename="package://jackal_description/meshes/novatel-smart6.stl"/>
+        <mesh filename="package://srd_pkg/jackal/jackal_description/meshes/novatel-smart6.stl"/>
       </geometry>
       <material name="novatel_white">

File: jackal/jackal_description/urdf/accessories/novatel_smart7.urdf.xacro (robot description, xacro)
@@ -6,5 +6,5 @@
         <origin xyz="-0.095 0 0" rpy="${pi/2} 0 -${pi/2}" />
         <geometry>
-          <mesh filename="package://jackal_description/meshes/novatel-smart7.stl"/>
+          <mesh filename="package://srd_pkg/jackal/jackal_description/meshes/novatel-smart7.stl"/>
         </geometry>
         <material name="novatel_white">
@@ -15,5 +15,5 @@
         <origin xyz="-0.095 0 0" rpy="${pi/2} 0 -${pi/2}" />
         <geometry>
-          <mesh filename="package://jackal_description/meshes/novatel-smart7.stl"/>
+          <mesh filename="package://srd_pkg/jackal/jackal_description/meshes/novatel-smart7.stl"/>
         </geometry>
       </collision>

File: jackal/jackal_description/urdf/accessories/sick_lms1xx_inverted_mount.urdf.xacro (robot description, xacro)
@@ -39,5 +39,5 @@
         <geometry>
           <!-- Origin of this mesh is the base of the bracket. -->
-          <mesh filename="package://jackal_description/meshes/sick-lms1xx-inverted-bracket.stl" />
+          <mesh filename="package://srd_pkg/jackal/jackal_description/meshes/sick-lms1xx-inverted-bracket.stl" />
         </geometry>
         <material name="dark_grey" />

File: jackal/jackal_description/urdf/accessories/sick_lms1xx_upright_mount.urdf.xacro (robot description, xacro)
@@ -39,5 +39,5 @@
         <geometry>
           <!-- Origin of this mesh is the base of the bracket. -->
-          <mesh filename="package://jackal_description/meshes/sick-lms1xx-upright-bracket.stl" />
+          <mesh filename="package://srd_pkg/jackal/jackal_description/meshes/sick-lms1xx-upright-bracket.stl" />
         </geometry>
         <material name="dark_grey" />

File: jackal/jackal_description/urdf/accessories/stereo_camera_mount.urdf.xacro (robot description, xacro)
@@ -6,5 +6,5 @@
         <origin xyz="0 0 0" rpy="0 0 0" />
         <geometry>
-          <mesh filename="package://jackal_description/meshes/stereo-camera-bracket.stl" />
+          <mesh filename="package://srd_pkg/jackal/jackal_description/meshes/stereo-camera-bracket.stl" />
         </geometry>
         <material name="dark_grey" />
@@ -15,5 +15,5 @@
         <origin xyz="0 0 0" rpy="0 0 0" />
         <geometry>
-          <mesh filename="package://jackal_description/meshes/stereo-camera-beam.stl" />
+          <mesh filename="package://srd_pkg/jackal/jackal_description/meshes/stereo-camera-beam.stl" />
         </geometry>
         <material name="dark_grey" />

File: jackal/jackal_description/urdf/jackal.urdf.xacro (robot description, xacro)
@@ -2,19 +2,20 @@
 <robot name="jackal" xmlns:xacro="http://www.ros.org/wiki/xacro">
   <xacro:property name="PI" value="3.1415926535897931" />
-  <xacro:property name="wheelbase" value="0.262" />
-  <xacro:property name="track" value="0.37559" />
-  <xacro:property name="wheel_vertical_offset" value="0.0345" />
-  <xacro:property name="footprint_vertical_offset" value="-0.0655" />
-  <xacro:property name="wheel_radius" value="0.098" />
-  <xacro:property name="wheel_width" value="0.040" />
-  <xacro:property name="chassis_length" value="0.420" />
-  <xacro:property name="chassis_width" value="0.310" />
-  <xacro:property name="chassis_height" value="0.184" />
-  <xacro:property name="dummy_inertia" value="1e-09"/>
-  <xacro:property name="mount_spacing" value="0.120" />
-  <material name="dark_grey"><color rgba="0.2 0.2 0.2 1.0" /></material>
-  <material name="light_grey"><color rgba="0.4 0.4 0.4 1.0" /></material>
-  <material name="yellow"><color rgba="0.8 0.8 0.0 1.0" /></material>
-  <material name="black"><color rgba="0.15 0.15 0.15 1.0" /></material>
+  <xacro:property name="wheelbase"                  value="0.262" />
+  <xacro:property name="track"                      value="0.37559" />
+  <xacro:property name="wheel_vertical_offset"      value="0.0345" />
+  <xacro:property name="footprint_vertical_offset"  value="-0.0655" />
+  <xacro:property name="wheel_radius"   value="0.098" />
+  <xacro:property name="wheel_width"    value="0.040" />
+  <xacro:property name="chassis_length"   value="0.420" />
+  <xacro:property name="chassis_width"    value="0.310" />
+  <xacro:property name="chassis_height"   value="0.184" />
+  <xacro:property name="dummy_inertia"    value="1e-09"/>
+  <xacro:property name="mount_spacing"    value="0.120" />
+  <!-- Define colors -->
+  <material name="dark_grey">   <color  rgba="0.2 0.2 0.2 1.0" />     </material>
+  <material name="light_grey">  <color  rgba="0.4 0.4 0.4 1.0" />     </material>
+  <material name="yellow">      <color  rgba="0.8 0.8 0.0 1.0" />     </material>
+  <material name="black">       <color  rgba="0.15 0.15 0.15 1.0" />  </material>
   <xacro:macro name="wheel" params="prefix *joint_pose">
     <link name="${prefix}_wheel_link">
@@ -22,5 +23,5 @@
         <origin xyz="0 0 0" rpy="${PI/2} 0 0"/>
         <geometry>
-          <mesh filename="package://jackal_description/meshes/jackal-wheel.stl"/>
+          <mesh filename="package://srd_pkg/jackal/jackal_description/meshes/jackal-wheel.stl"/>
         </geometry>
         <material name="black" />
@@ -90,5 +91,5 @@
       <origin xyz="0 0 ${footprint_vertical_offset}" rpy="${PI/2} 0 ${PI/2}"/>
       <geometry>
-        <mesh filename="package://jackal_description/meshes/jackal-base.stl"/>
+        <mesh filename="package://srd_pkg/jackal/jackal_description/meshes/jackal-base.stl"/>
       </geometry>
       <material name="dark_grey" />
@@ -115,5 +116,5 @@
       <visual>
         <geometry>
-          <mesh filename="package://jackal_description/meshes/jackal-fender.stl"/>
+          <mesh filename="package://srd_pkg/jackal/jackal_description/meshes/jackal-fender.stl"/>
         </geometry>
         <material name="yellow" />
@@ -125,5 +126,5 @@
       <visual>
         <geometry>
-          <mesh filename="package://jackal_description/meshes/accessory_fender.stl"/>
+          <mesh filename="package://srd_pkg/jackal/jackal_description/meshes/accessory_fender.stl"/>
         </geometry>
         <material name="yellow" />
@@ -146,5 +147,5 @@
       <visual>
         <geometry>
-          <mesh filename="package://jackal_description/meshes/jackal-fender.stl"/>
+          <mesh filename="package://srd_pkg/jackal/jackal_description/meshes/jackal-fender.stl"/>
         </geometry>
         <material name="yellow" />
@@ -156,5 +157,5 @@
       <visual>
         <geometry>
-          <mesh filename="package://jackal_description/meshes/accessory_fender.stl"/>
+          <mesh filename="package://srd_pkg/jackal/jackal_description/meshes/accessory_fender.stl"/>
         </geometry>
         <material name="yellow" />
@@ -219,9 +220,9 @@
   </joint>
   <!-- Bring in simulation data for Gazebo. -->
-  <xacro:include filename="$(find jackal_description)/urdf/jackal.gazebo" />
+  <xacro:include filename="$(find srd_pkg)/jackal/jackal_description/urdf/jackal.gazebo" />
   <!-- Optional standard accessories, including their simulation data. The rendering
        of these into the final description is controlled by optenv variables, which
        default each one to off.-->
-  <xacro:include filename="$(find jackal_description)/urdf/accessories.urdf.xacro" />
+  <xacro:include filename="$(find srd_pkg)/jackal/jackal_description/urdf/accessories.urdf.xacro" />
   <!-- OutdoorNav -->
   <xacro:arg name="outdoornav_enabled"       default="$(optenv OUTDOORNAV_ENABLED 0)" />

Commit message: LMS1XX funzionante (testato solo con un robot)
- Jackal multipli con namespace differenti
- AMCL all'interno del namespace che si collega al topic /map condiviso
- LSM1XX funzionante con questo setup (testato solo su un robot)

File: jackal/jackal_description/urdf/accessories.urdf.xacro (robot description, xacro)
@@ -261,8 +261,8 @@
   <!-- If enabled, generate the flea3 camera payload with a tilt of 30 degrees. -->
   <xacro:if value="$(optenv JACKAL_FLEA3 0)">
-    <xacro:property name="name" value="$(optenv JACKAL_FLEA3_NAME front)" />
-    <xacro:property name="tilt" value="$(optenv JACKAL_FLEA3_TILT 0.5236)" />
-    <xacro:property name="tower" value="$(optenv JACKAL_FLEA3_TOWER 1)" />
-    <xacro:property name="mount" value="$(optenv JACKAL_FLEA3_MOUNT front)" />
+    <xacro:property name="name"   value="$(optenv JACKAL_FLEA3_NAME front)" />
+    <xacro:property name="tilt"   value="$(optenv JACKAL_FLEA3_TILT 0.5236)" />
+    <xacro:property name="tower"  value="$(optenv JACKAL_FLEA3_TOWER 1)" />
+    <xacro:property name="mount"  value="$(optenv JACKAL_FLEA3_MOUNT front)" />
     <xacro:property name="prefix" value="$(optenv JACKAL_FLEA3_PREFIX ${mount})" />
     <xacro:property name="parent" value="$(optenv JACKAL_FLEA3_PARENT ${mount}_mount)" />

File: jackal/jackal_description/urdf/accessories/sick_lms1xx_upright_mount.urdf.xacro (robot description, xacro)
@@ -28,5 +28,5 @@
   <xacro:include filename="$(find lms1xx)/urdf/sick_lms1xx.urdf.xacro" />
   <xacro:macro name="sick_lms1xx_upright_mount" params="prefix topic parent_link *origin">
-    <xacro:sick_lms1xx frame="${prefix}_laser" topic="${topic}" />
+    <xacro:sick_lms1xx frame="${prefix}_laser" topic="${topic}" robot_namespace="$(arg namespace)" />
     <joint name="${prefix}_laser_mount_joint" type="fixed">
       <xacro:insert_block name="origin" />

File: jackal/jackal_description/urdf/jackal.urdf.xacro (robot description, xacro)
@@ -13,4 +13,5 @@
   <xacro:property name="dummy_inertia"    value="1e-09"/>
   <xacro:property name="mount_spacing"    value="0.120" />
+  <xacro:property name="camera_link"    value="0.05" />
   <!-- Define colors -->
   <material name="dark_grey">   <color  rgba="0.2 0.2 0.2 1.0" />     </material>
@@ -18,4 +19,5 @@
   <material name="yellow">      <color  rgba="0.8 0.8 0.0 1.0" />     </material>
   <material name="black">       <color  rgba="0.15 0.15 0.15 1.0" />  </material>
+  <material name="red">         <color  rgba="0.8 0.0 0.0 1.0" />     </material>
   <xacro:macro name="wheel" params="prefix *joint_pose">
     <link name="${prefix}_wheel_link">
@@ -219,4 +221,6 @@
     <origin xyz="${mount_spacing} 0 0" />
   </joint>
+  <!-- Adding custom camera -->
+  <!-- <xacro:include filename="accessories/custom_camera.urdf.xacro" /> -->
   <!-- Bring in simulation data for Gazebo. -->
   <xacro:include filename="$(find srd_pkg)/jackal/jackal_description/urdf/jackal.gazebo" />
@@ -224,16 +228,12 @@
        of these into the final description is controlled by optenv variables, which
        default each one to off.-->
-  <xacro:include filename="$(find srd_pkg)/jackal/jackal_description/urdf/accessories.urdf.xacro" />
+  <xacro:include  filename="$(find srd_pkg)/jackal/jackal_description/urdf/accessories.urdf.xacro" />
   <!-- OutdoorNav -->
-  <xacro:arg name="outdoornav_enabled"       default="$(optenv OUTDOORNAV_ENABLED 0)" />
-  <xacro:arg name="outdoornav_configuration" default="$(optenv OUTDOORNAV_CONFIGURATION standard)" />
+  <!-- <xacro:arg name="outdoornav_enabled"       default="$(optenv OUTDOORNAV_ENABLED 0)" />
+  <xacro:arg name="outdoornav_configuration" default="$(optenv OUTDOORNAV_CONFIGURATION standard)" /> -->
   <!-- OutdoorNav URDF Config -->
-  <xacro:if value="$(arg outdoornav_enabled)">
+  <!-- <xacro:if value="$(arg outdoornav_enabled)">
     <xacro:include filename="$(find cpr_onav_description)/urdf/outdoornav_description.urdf.xacro" />
     <xacro:outdoornav_sensors outdoornav_configuration="$(arg outdoornav_configuration)" />
-  </xacro:if>
-  <!-- Optional custom includes. -->
-  <xacro:include filename="$(optenv JACKAL_URDF_EXTRAS empty.urdf)" />
-  <!-- Optional for Clearpath internal softwares -->
-  <xacro:include filename="$(optenv CPR_URDF_EXTRAS empty.urdf)" />
+  </xacro:if> -->
 </robot>
