Commit message: Modifiche varie

File: jackal/jackal_description/urdf/accessories.urdf.xacro (robot description, xacro)
@@ -14,5 +14,5 @@
   <xacro:include filename="$(find srd_pkg)/jackal/jackal_description/urdf/accessories/bridge_plate.urdf.xacro" />
   <!-- 2D Lidars -->
-  <xacro:include filename="$(find sick_tim)/urdf/sick_tim.urdf.xacro" />
+  <xacro:include filename="$(find srd_pkg)/include/sick_tim/urdf/sick_tim.urdf.xacro" />
   <xacro:include filename="$(find srd_pkg)/include/lms1xx/urdf/sick_lms1xx.urdf.xacro" />
   <xacro:include filename="$(find srd_pkg)/jackal/jackal_description/urdf/accessories/sick_lms1xx_inverted_mount.urdf.xacro" />
@@ -88,5 +88,5 @@
     <xacro:if value="${lidar_model == 'tim551'}">
       <xacro:property name="prefix" value="$(optenv JACKAL_LASER_PREFIX tim551)" />
-      <xacro:sick_tim551 name="${prefix}" ros_topic="${topic}"/>
+      <xacro:sick_tim551 name="${prefix}" ros_topic="${topic}" robot_namespace="$(arg namespace)"/>
       <joint name="${prefix}_mount_link_joint" type="fixed">
         <origin xyz="$(optenv JACKAL_LASER_OFFSET 0 0 0)" rpy="$(optenv JACKAL_LASER_RPY 0 0 0)"/>
@@ -261,8 +261,8 @@
   <!-- If enabled, generate the flea3 camera payload with a tilt of 30 degrees. -->
   <xacro:if value="$(optenv JACKAL_FLEA3 0)">
-    <xacro:property name="name"   value="$(optenv JACKAL_FLEA3_NAME front)" />
-    <xacro:property name="tilt"   value="$(optenv JACKAL_FLEA3_TILT 0.5236)" />
-    <xacro:property name="tower"  value="$(optenv JACKAL_FLEA3_TOWER 1)" />
-    <xacro:property name="mount"  value="$(optenv JACKAL_FLEA3_MOUNT front)" />
+    <xacro:property name="name" value="$(optenv JACKAL_FLEA3_NAME front)" />
+    <xacro:property name="tilt" value="$(optenv JACKAL_FLEA3_TILT 0.5236)" />
+    <xacro:property name="tower" value="$(optenv JACKAL_FLEA3_TOWER 1)" />
+    <xacro:property name="mount" value="$(optenv JACKAL_FLEA3_MOUNT front)" />
     <xacro:property name="prefix" value="$(optenv JACKAL_FLEA3_PREFIX ${mount})" />
     <xacro:property name="parent" value="$(optenv JACKAL_FLEA3_PARENT ${mount}_mount)" />
@@ -399,9 +399,10 @@
     <xacro:if value="$(optenv JACKAL_FRONT_FENDER_UST10 0)">
       <xacro:hokuyo_ust10_mount
-        prefix="front"
+        prefix="fender"
         parent_link="front_fender_accessory_link"
-        min_angle="${-pi/2}"
-        max_angle="${pi/2}"
-        topic="$(optenv JACKAL_FRONT_LASER_TOPIC front/scan)">
+        min_angle="${-pi*7/13}"
+        max_angle="${pi*7/13}"
+        topic="fender/scan"
+        robot_namespace="$(arg namespace)" >
         <origin xyz="0 0 0" rpy="0 0 0" />
       </xacro:hokuyo_ust10_mount>

File: jackal/jackal_description/urdf/accessories/hokuyo_ust10.urdf.xacro (robot description, xacro)
@@ -1,7 +1,7 @@
 <?xml version="1.0"?>
 <robot xmlns:xacro="http://ros.org/wiki/xacro">
-  <xacro:macro name="hokuyo_ust10_mount" params="prefix topic parent_link min_angle:=-2.35619 max_angle:=2.35619 *origin">
+  <xacro:macro name="hokuyo_ust10_mount" params="prefix topic parent_link min_angle:=-2.35619 max_angle:=2.35619 *origin robot_namespace:=/">
     <xacro:macro name="hokuyo_ust10" params="frame:=laser topic:=scan sample_size:=720 update_rate:=50
-               min_angle:=-2.35619 max_angle:=2.35619 min_range:=0.1 max_range:=30.0 robot_namespace:=/">
+                                             min_range:=0.1 max_range:=30.0 robot_namespace:=/">
       <link name="${frame}">
         <inertial>
@@ -14,5 +14,5 @@
       </link>
       <gazebo reference="${frame}">
-        <turnGravityOff>true</turnGravityOff>
+        <turnGravityOff>false</turnGravityOff>
         <sensor type="ray" name="${frame}">
           <pose>0 0 0 0 0 0</pose>
@@ -41,5 +41,5 @@
           <plugin name="gazebo_ros_laser" filename="libgazebo_ros_laser.so">
             <topicName>${topic}</topicName>
-            <frameName>${frame}</frameName>
+            <frameName>${robot_namespace}/${frame}</frameName>
             <robotNamespace>${robot_namespace}</robotNamespace>
           </plugin>
@@ -47,5 +47,5 @@
       </gazebo>
     </xacro:macro>
-    <xacro:hokuyo_ust10 frame="${prefix}_laser" topic="${topic}"/>
+    <xacro:hokuyo_ust10 frame="${prefix}_laser" topic="${topic}" robot_namespace="$(arg namespace)" />
     <joint name="${prefix}_laser_mount_joint" type="fixed">
       <xacro:insert_block name="origin" />

File: jackal/jackal_description/urdf/accessories/sick_lms1xx_inverted_mount.urdf.xacro (robot description, xacro)
@@ -1,28 +1,3 @@
 <?xml version="1.0"?>
-<!--
-Copyright (c) 2013, Goncalo Cabrita, ISR University of Coimbra
-Copyright (c) 2014, 2015 Clearpath Robotics
-All rights reserved.
-Redistribution and use in source and binary forms, with or without
-modification, are permitted provided that the following conditions are met:
-    * Redistributions of source code must retain the above copyright
-      notice, this list of conditions and the following disclaimer.
-    * Redistributions in binary form must reproduce the above copyright
-      notice, this list of conditions and the following disclaimer in the
-      documentation and/or other materials provided with the distribution.
-    * Neither the name of Clearpath Robotics nor the
-      names of its contributors may be used to endorse or promote products
-      derived from this software without specific prior written permission.
-THIS SOFTWARE IS PROVIDED BY THE COPYRIGHT HOLDERS AND CONTRIBUTORS "AS IS" AND
-ANY EXPRESS OR IMPLIED WARRANTIES, INCLUDING, BUT NOT LIMITED TO, THE IMPLIED
-WARRANTIES OF MERCHANTABILITY AND FITNESS FOR A PARTICULAR PURPOSE ARE
-DISCLAIMED. IN NO EVENT SHALL THE COPYRIGHT HOLDERS BE LIABLE FOR ANY
-DIRECT, INDIRECT, INCIDENTAL, SPECIAL, EXEMPLARY, OR CONSEQUENTIAL DAMAGES
-(INCLUDING, BUT NOT LIMITED TO, PROCUREMENT OF SUBSTITUTE GOODS OR SERVICES;
-LOSS OF USE, DATA, OR PROFITS; OR BUSINESS INTERRUPTION) HOWEVER CAUSED AND
-ON ANY THEORY OF LIABILITY, WHETHER IN CONTRACT, STRICT LIABILITY, OR TORT
-(INCLUDING NEGLIGENCE OR OTHERWISE) ARISING IN ANY WAY OUT OF THE USE OF THIS
-SOFTWARE, EVEN IF ADVISED OF THE POSSIBILITY OF SUCH DAMAGE.
--->
 <robot xmlns:xacro="http://www.ros.org/wiki/xacro">
   <xacro:include filename="$(find srd_pkg)/include/lms1xx/urdf/sick_lms1xx.urdf.xacro" />
@@ -38,5 +13,4 @@
         <origin xyz="0 0 0" rpy="0 0 0" />
         <geometry>
-          <!-- Origin of this mesh is the base of the bracket. -->
           <mesh filename="package://srd_pkg/jackal/jackal_description/meshes/sick-lms1xx-inverted-bracket.stl" />
         </geometry>
@@ -45,5 +19,4 @@
     </link>
     <joint name="${prefix}_laser_joint" type="fixed">
-      <!-- This offset is from the base of the bracket to the LIDAR's focal point. -->
       <origin xyz="0.04 0 0.066" rpy="3.141592 0 0" />
       <parent link="${prefix}_laser_mount" />

File: jackal/jackal_description/urdf/accessories/sick_lms1xx_upright_mount.urdf.xacro (robot description, xacro)
@@ -1,28 +1,3 @@
 <?xml version="1.0"?>
-<!--
-Copyright (c) 2013, Goncalo Cabrita, ISR University of Coimbra
-Copyright (c) 2014, 2015 Clearpath Robotics
-All rights reserved.
-Redistribution and use in source and binary forms, with or without
-modification, are permitted provided that the following conditions are met:
-    * Redistributions of source code must retain the above copyright
-      notice, this list of conditions and the following disclaimer.
-    * Redistributions in binary form must reproduce the above copyright
-      notice, this list of conditions and the following disclaimer in the
-      documentation and/or other materials provided with the distribution.
-    * Neither the name of Clearpath Robotics nor the
-      names of its contributors may be used to endorse or promote products
-      derived from this software without specific prior written permission.
-THIS SOFTWARE IS PROVIDED BY THE COPYRIGHT HOLDERS AND CONTRIBUTORS "AS IS" AND
-ANY EXPRESS OR IMPLIED WARRANTIES, INCLUDING, BUT NOT LIMITED TO, THE IMPLIED
-WARRANTIES OF MERCHANTABILITY AND FITNESS FOR A PARTICULAR PURPOSE ARE
-DISCLAIMED. IN NO EVENT SHALL THE COPYRIGHT HOLDERS BE LIABLE FOR ANY
-DIRECT, INDIRECT, INCIDENTAL, SPECIAL, EXEMPLARY, OR CONSEQUENTIAL DAMAGES
-(INCLUDING, BUT NOT LIMITED TO, PROCUREMENT OF SUBSTITUTE GOODS OR SERVICES;
-LOSS OF USE, DATA, OR PROFITS; OR BUSINESS INTERRUPTION) HOWEVER CAUSED AND
-ON ANY THEORY OF LIABILITY, WHETHER IN CONTRACT, STRICT LIABILITY, OR TORT
-(INCLUDING NEGLIGENCE OR OTHERWISE) ARISING IN ANY WAY OUT OF THE USE OF THIS
-SOFTWARE, EVEN IF ADVISED OF THE POSSIBILITY OF SUCH DAMAGE.
--->
 <robot xmlns:xacro="http://www.ros.org/wiki/xacro">
   <xacro:include filename="$(find srd_pkg)/include/lms1xx/urdf/sick_lms1xx.urdf.xacro" />
@@ -38,5 +13,4 @@
         <origin xyz="0 0 0" rpy="0 0 0" />
         <geometry>
-          <!-- Origin of this mesh is the base of the bracket. -->
           <mesh filename="package://srd_pkg/jackal/jackal_description/meshes/sick-lms1xx-upright-bracket.stl" />
         </geometry>
@@ -45,5 +19,4 @@
     </link>
     <joint name="${prefix}_laser_joint" type="fixed">
-      <!-- This offset is from the base of the bracket to the LIDAR's focal point. -->
       <origin xyz="0 0 0.149" rpy="0 0 0" />
       <parent link="${prefix}_laser_mount" />

File: jackal/jackal_description/urdf/jackal.urdf.xacro (robot description, xacro)
@@ -1,23 +1,25 @@
 <?xml version="1.0"?>
 <robot name="jackal" xmlns:xacro="http://www.ros.org/wiki/xacro">
-  <xacro:property name="PI" value="3.1415926535897931" />
-  <xacro:property name="wheelbase"                  value="0.262" />
-  <xacro:property name="track"                      value="0.37559" />
-  <xacro:property name="wheel_vertical_offset"      value="0.0345" />
-  <xacro:property name="footprint_vertical_offset"  value="-0.0655" />
-  <xacro:property name="wheel_radius"   value="0.098" />
-  <xacro:property name="wheel_width"    value="0.040" />
-  <xacro:property name="chassis_length"   value="0.420" />
-  <xacro:property name="chassis_width"    value="0.310" />
-  <xacro:property name="chassis_height"   value="0.184" />
-  <xacro:property name="dummy_inertia"    value="1e-09"/>
-  <xacro:property name="mount_spacing"    value="0.120" />
-  <xacro:property name="camera_link"    value="0.05" />
-  <!-- Define colors -->
-  <material name="dark_grey">   <color  rgba="0.2 0.2 0.2 1.0" />     </material>
-  <material name="light_grey">  <color  rgba="0.4 0.4 0.4 1.0" />     </material>
-  <material name="yellow">      <color  rgba="0.8 0.8 0.0 1.0" />     </material>
-  <material name="black">       <color  rgba="0.15 0.15 0.15 1.0" />  </material>
-  <material name="red">         <color  rgba="0.8 0.0 0.0 1.0" />     </material>
+  <xacro:property name="PI"                           value="3.1415926535897931" />
+  <xacro:property name="wheelbase"                    value="0.262" />
+  <xacro:property name="track"                        value="0.37559" />
+  <xacro:property name="wheel_vertical_offset"        value="0.0345" />
+  <xacro:property name="footprint_vertical_offset"    value="-0.0655" />
+  <!-- Geometria ruote -->
+  <xacro:property name="wheel_radius"                 value="0.098" />
+  <xacro:property name="wheel_width"                  value="0.040" />
+  <xacro:property name="mount_spacing"                value="0.120" />
+  <!-- Geometria corpo centrale -->
+  <xacro:property name="chassis_length"               value="0.420" />
+  <xacro:property name="chassis_width"                value="0.310" />
+  <xacro:property name="chassis_height"               value="0.184" />
+  <!-- Inerzia fasulla per non usare un valore nullo -->
+  <xacro:property name="dummy_inertia"                value="1e-09"/>
+  <!-- Colori -->
+  <material name="dark_grey">   <color    rgba="0.2 0.2 0.2 1.0" />     </material>
+  <material name="light_grey">  <color    rgba="0.4 0.4 0.4 1.0" />     </material>
+  <material name="yellow">      <color    rgba="0.8 0.8 0.0 1.0" />     </material>
+  <material name="black">       <color    rgba="0.15 0.15 0.15 1.0" />  </material>
+  <!-- Macro per definire le 4 ruote, che verrà richiamata successivamente -->
   <xacro:macro name="wheel" params="prefix *joint_pose">
     <link name="${prefix}_wheel_link">
@@ -53,4 +55,5 @@
       <fdir1 value="1 0 0"/>
     </gazebo>
+    <!-- Joint tra corpo centrale e ruota -->
     <joint name="${prefix}_wheel" type="continuous">
       <parent link="chassis_link"/>
@@ -71,4 +74,5 @@
     </transmission>
   </xacro:macro>
+  <!-- La macro definita prima viene richiamata per ogni ruota -->
   <xacro:wheel prefix="front_left">
     <origin xyz="${wheelbase/2} ${track/2} ${wheel_vertical_offset}" rpy="0 0 0" />
@@ -84,4 +88,5 @@
   </xacro:wheel>
   <link name="base_link"></link>
+  <!-- Joint tra base_link e copro centrale -->
   <joint name="base_link_joint" type="fixed">
     <origin xyz="0 0 0" rpy="0 0 0" />
@@ -89,4 +94,5 @@
     <child link="chassis_link" />
   </joint>
+  <!-- Link del corpo centrale -->
   <link name="chassis_link">
     <visual>
@@ -114,4 +120,5 @@
       </inertial>
   </link>
+  <!-- Prafango anteriore senza portaoggetti -->
   <xacro:unless value="$(optenv JACKAL_FRONT_ACCESSORY_FENDER 0)">
     <link name="front_fender_link">
@@ -124,4 +131,23 @@
     </link>
   </xacro:unless>
+  <!-- Parafango anteriore con portaoggetti -->
+  <xacro:if value="$(optenv JACKAL_FRONT_ACCESSORY_FENDER 0)">
+    <link name="front_fender_link">
+      <visual>
+        <geometry>
+          <mesh filename="package://srd_pkg/jackal/jackal_description/meshes/accessory_fender.stl"/>
+        </geometry>
+        <material name="yellow" />
+      </visual>
+    </link>
+    <!-- Nuovo link e joint per accessori anteriori -->
+    <link name="front_fender_accessory_link"/>
+    <joint name="front_fender_accessory_joint" type="fixed">
+      <origin xyz="0.25629 0 0.07455" rpy="${PI} 0 0" />
+      <parent link="front_fender_link" />
+      <child link="front_fender_accessory_link" />
+    </joint>
+  </xacro:if>
+  <!-- Joint tra corpo centrale e parafango anteriore -->
   <joint name="front_fender_joint" type="fixed">
     <origin xyz="0 0 0" rpy="0 0 0"/>
@@ -129,4 +155,5 @@
     <child link="front_fender_link" />
   </joint>
+  <!-- Parafango posteriore senza portaoggetti -->
   <xacro:unless value="$(optenv JACKAL_REAR_ACCESSORY_FENDER 0)">
     <link name="rear_fender_link">
@@ -139,4 +166,23 @@
     </link>
   </xacro:unless>
+  <!-- Parafango posteriore con portaoggetti -->
+  <xacro:if value="$(optenv JACKAL_REAR_ACCESSORY_FENDER 0)">
+    <link name="rear_fender_link">
+      <visual>
+        <geometry>
+          <mesh filename="package://jackal_description/meshes/accessory_fender.stl"/>
+        </geometry>
+        <material name="yellow" />
+      </visual>
+    </link>
+    <!-- Nuovo link e joint per accessori posteriori -->
+    <link name="rear_fender_accessory_link"/>
+    <joint name="rear_fender_accessory_joint" type="fixed">
+      <origin xyz="0.25629 0 0.07455" rpy="${PI} 0 0" />
+      <parent link="rear_fender_link" />
+      <child link="rear_fender_accessory_link" />
+    </joint>
+  </xacro:if>
+  <!-- Joint tra corpo centrale e parafango posteriore -->
   <joint name="rear_fender_joint" type="fixed">
     <origin xyz="0 0 0" rpy="0 0 ${PI}"/>
@@ -171,4 +217,6 @@
     <origin xyz="-0.180 0.126 0.1815" />
   </joint>
+  <!-- Link e joint per montaggio centrale, a cui si collegano montaggio
+        anteriore e posteriore -->
   <link name="mid_mount"></link>
   <joint name="mid_mount_joint" type="fixed">
@@ -177,4 +225,5 @@
     <origin xyz="0 0 ${chassis_height}" />
   </joint>
+  <!-- Montaggio posteriore con joint al montaggio centrale -->
   <link name="rear_mount"></link>
   <joint name="rear_mount_joint" type="fixed">
@@ -183,4 +232,5 @@
     <origin xyz="${-mount_spacing} 0 0" />
   </joint>
+  <!-- Montaggio anteriore con joint al montaggio centrale -->
   <link name="front_mount"></link>
   <joint name="front_mount_joint" type="fixed">
@@ -190,5 +240,5 @@
   </joint>
   <!-- Adding custom camera -->
-  <xacro:include filename="accessories/custom_camera.urdf.xacro" />
+  <!-- <xacro:include filename="accessories/custom_camera.urdf.xacro" /> -->
   <!-- Bring in simulation data for Gazebo. -->
   <xacro:include filename="$(find srd_pkg)/jackal/jackal_description/urdf/jackal.gazebo" />
